File: MotorFreaker/FreakHat/FreakHat.kicad_pcb (KiCad board)
At the start: 2 copper layers, 7 parts, among them J1 DIN-5, J2 DIN-5, U1 74HC244, U2 74HC244, U4 LM7805_TO220

Commit message: hat
Parts:
- added RN1: 8 x 10K, Resistor_THT:R_Array_SIP8, F.Cu at (94.5, 36.3)
Connections:
- A1 pad D11: unconnected-(A1-PadD11) -> /DOUT
- A1 pad D13: unconnected-(A1-PadD13) -> /CLK
- A1 pad D2: unconnected-(A1-D2_INT0-PadD2) -> /CS_1
- A1 pad D3: unconnected-(A1-D3_INT1-PadD3) -> /CS_2
- A1 pad D4: unconnected-(A1-PadD4) -> /CS_3
- A1 pad D5: unconnected-(A1-PadD5) -> /CS_4
- A1 pad D6: unconnected-(A1-PadD6) -> /CS_5
- A1 pad D7: unconnected-(A1-PadD7) -> /CS_6
- A1 pad D8: unconnected-(A1-PadD8) -> /CS_7
- A1 pad D9: unconnected-(A1-PadD9) -> /CS_8
- U1 pad 11: unconnected-(U1-2A3-Pad11) -> /CLK
- U1 pad 13: unconnected-(U1-2A2-Pad13) -> /DOUT
- U1 pad 15: unconnected-(U1-2A1-Pad15) -> /CLK
- U1 pad 17: unconnected-(U1-2A0-Pad17) -> /DOUT
- U1 pad 2: unconnected-(U1-1A0-Pad2) -> /DOUT
- U1 pad 4: unconnected-(U1-1A1-Pad4) -> /CLK
- U1 pad 6: unconnected-(U1-1A2-Pad6) -> /DOUT
- U1 pad 8: unconnected-(U1-1A3-Pad8) -> /CLK
- U2 pad 11: unconnected-(U2-2A3-Pad11) -> /CLK
- U2 pad 13: unconnected-(U2-2A2-Pad13) -> /DOUT
- U2 pad 15: unconnected-(U2-2A1-Pad15) -> /CLK
- U2 pad 17: unconnected-(U2-2A0-Pad17) -> /DOUT
- U2 pad 2: unconnected-(U2-1A0-Pad2) -> /DOUT
- U2 pad 4: unconnected-(U2-1A1-Pad4) -> /CLK
- U2 pad 6: unconnected-(U2-1A2-Pad6) -> /DOUT
- U2 pad 8: unconnected-(U2-1A3-Pad8) -> /CLK
