File: MotorFreaker/FreakHat/FreakHat.kicad_pcb (KiCad board)
At the start: 2 copper layers, 17 parts, among them J1 DIN-5, J10 Conn_01x05, J2 DIN-5, J4 Conn_01x05, J5 Conn_01x05, J6 Conn_01x05, J7 Conn_01x05, J8 Conn_01x05, J9 Conn_01x05, U1 74HC244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

Commit message: midi
Parts:
- removed the J1 at (33.9, 54.0)
- removed the J2 at (51.3, 54.0)
- removed REF**: JST_XH_B5B-XH-AM_1x05_P2.50mm_Vertical, Connector_JST:JST_XH_B5B-XH-AM_1x05_P2.50mm_Vertical
- removed RN1: 8 x 10K, Resistor_THT:R_Array_SIP9
- removed U3: 6N138, Package_DIP:DIP-8_W7.62mm_Socket
- removed U5: SN7407N, Package_DIP:DIP-14_W7.62mm_Socket
- added C1: 0.1uF, Capacitor_THT:C_Disc_D3.4mm_W2.1mm_P2.50mm, F.Cu at (85.1, 110.3)
- added C2: 0.1uF, Capacitor_THT:C_Disc_D3.4mm_W2.1mm_P2.50mm, F.Cu at (85.1, 92.5)
- added C3: 10uF, Capacitor_THT:CP_Radial_D5.0mm_P2.00mm, F.Cu at (84.6, 126.2)
- added C4: 100uF, Capacitor_THT:CP_Radial_D8.0mm_P3.50mm, F.Cu at (66.2, 123.4)
- added C5: 0.1uF, Capacitor_THT:C_Disc_D3.4mm_W2.1mm_P2.50mm, F.Cu at (72.6, 130.0)
- added J10: Conn_01x02, Connector_Molex:Molex_KK-254_AE-6410-02A_1x02_P2.54mm_Vertical, F.Cu at (109.7, 124.5)
- added J11: Conn_01x02, Connector_Molex:Molex_KK-254_AE-6410-02A_1x02_P2.54mm_Vertical, F.Cu at (117.3, 124.5)
- added J12: Conn_01x02, Connector_Molex:Molex_KK-254_AE-6410-02A_1x02_P2.54mm_Vertical, F.Cu at (121.9, 115.3)
- added J7: Conn_01x05, Connector_Molex:Molex_KK-254_AE-6410-05A_1x05_P2.54mm_Vertical, F.Cu at (98.8, 116.1)
- added J9: Conn_01x04, Connector_Molex:Molex_KK-254_AE-6410-04A_1x04_P2.54mm_Vertical, F.Cu at (122.2, 98.8)
- added SW1: SW_DIP_x02, Button_Switch_THT:SW_DIP_SPSTx02_Slide_9.78x7.26mm_W7.62mm_P2.54mm, F.Cu at (100.6, 125.7)
- J1: renamed from J5; footprint Connector_JST:JST_XH_B5B-XH-AM_1x05_P2.50mm_Vertical -> Connector_Molex:Molex_KK-254_AE-6410-05A_1x05_P2.54mm_Vertical
- J2: renamed from J6; footprint Connector_JST:JST_XH_B5B-XH-AM_1x05_P2.50mm_Vertical -> Connector_Molex:Molex_KK-254_AE-6410-05A_1x05_P2.54mm_Vertical
- J3: renamed from J7; footprint Connector_JST:JST_XH_B5B-XH-AM_1x05_P2.50mm_Vertical -> Connector_Molex:Molex_KK-254_AE-6410-05A_1x05_P2.54mm_Vertical
- J4: renamed from J8; footprint Connector_JST:JST_XH_B5B-XH-AM_1x05_P2.50mm_Vertical -> Connector_Molex:Molex_KK-254_AE-6410-05A_1x05_P2.54mm_Vertical
- J5: renamed from J9; footprint Connector_JST:JST_XH_B5B-XH-AM_1x05_P2.50mm_Vertical -> Connector_Molex:Molex_KK-254_AE-6410-05A_1x05_P2.54mm_Vertical
- J6: renamed from J10; footprint Connector_JST:JST_XH_B5B-XH-AM_1x05_P2.50mm_Vertical -> Connector_Molex:Molex_KK-254_AE-6410-05A_1x05_P2.54mm_Vertical
- J8: renamed from J4; footprint Connector_JST:JST_XH_B5B-XH-AM_1x05_P2.50mm_Vertical -> Connector_Molex:Molex_KK-254_AE-6410-05A_1x05_P2.54mm_Vertical
- moved J5 89.5 mm to (98.8, 107.2), turned to 180 degrees
- moved J3 88.4 mm to (98.8, 98.3), turned to 180 degrees
- moved J1 87.7 mm to (98.8, 89.2), turned to 180 degrees
- moved J8 78.6 mm to (113.3, 116.1), turned to 180 degrees
- moved J6 77.8 mm to (113.3, 107.2), turned to 180 degrees
- moved U1 77.2 mm to (81.8, 89.4), turned to -90 degrees
- moved J4 75.7 mm to (113.3, 98.3), turned to 180 degrees
- moved J2 74.3 mm to (113.3, 89.2), turned to 180 degrees
- moved U4 71.9 mm to (77.7, 123.4), turned to 180 degrees
- moved U2 70.0 mm to (81.8, 107.7), turned to -90 degrees
Connections:
- A1 pad A0: /DIP_2 -> /DIP_1
- A1 pad A1: /DIP_1 -> /DIP_2
- A1 pad A2: unconnected-(A1-PadA2) -> /SW_1
- A1 pad A3: unconnected-(A1-PadA3) -> /SW_2
- A1 pad A4: unconnected-(A1-PadA4) -> /SW_3
- A1 pad D1: unconnected-(A1-D1/TX-PadD1) -> Net-(A1-D1/TX)
- A1 pad D2: /CS_1 -> /CS_8
- A1 pad D3: /CS_2 -> /CS_6
- A1 pad D4: /CS_3 -> /CS_4
- A1 pad D5: /CS_4 -> /CS_2
- A1 pad D6: /CS_5 -> /CS_7
- A1 pad D7: /CS_6 -> /CS_5
- A1 pad D8: /CS_7 -> /CS_3
- A1 pad D9: /CS_8 -> /CS_1
- A1 pad VIN: +5V -> +9V
- U1 pad 12: /CLK_2 -> /CLK_4
- U1 pad 14: /DOUT_2 -> /DOUT_4
- U1 pad 16: /CLK_1 -> /CLK_3
- U1 pad 18: /DOUT_1 -> /DOUT_3
- U1 pad 3: /DOUT_3 -> /DOUT_1
- U1 pad 5: /CLK_3 -> /CLK_1
- U1 pad 7: /DOUT_4 -> /DOUT_2
- U1 pad 9: /CLK_4 -> /CLK_2
- U2 pad 12: /CLK_6 -> /CLK_8
- U2 pad 14: /DOUT_6 -> /DOUT_8
- U2 pad 16: /CLK_5 -> /CLK_7
- U2 pad 18: /DOUT_5 -> /DOUT_7
- U2 pad 3: /DOUT_7 -> /DOUT_5
- U2 pad 5: /CLK_7 -> /CLK_5
- U2 pad 7: /DOUT_8 -> /DOUT_6
- U2 pad 9: /CLK_8 -> /CLK_6
Routing:
- net +5V: track 0.00 -> 154.5 mm
- net /DOUT: track 0.00 -> 88.5 mm
- net /CLK: track 0.00 -> 88.5 mm
- net /CLK_8: track 0.00 -> 51.5 mm
- net /CLK_6: track 0.00 -> 50.5 mm
- net /CLK_2: track 0.00 -> 50.4 mm
- net /CLK_4: track 0.00 -> 50.1 mm
- net /CS_7: track 0.00 -> 42.7 mm
- net /DOUT_8: track 0.00 -> 42.6 mm
- net /DOUT_6: track 0.00 -> 42.5 mm
- net /DOUT_2: track 0.00 -> 42.4 mm
- net /DOUT_4: track 0.00 -> 42.1 mm
- net /CS_8: track 0.00 -> 38.4 mm
- net /CS_5: track 0.00 -> 32.7 mm
- net /CS_6: track 0.00 -> 28.4 mm
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- added copper zone on B.Cu, net GND
- added copper zone on F.Cu, net GND
Other:
- board outline added: 69.1 x 53.3 mm
- board text added: "1"
- board text added: "2"
- board text added: "3"
- board text added: "4"
- board text added: "5"
- board text added: "5V"
- board text added: "6"
- board text added: "7"
- board text added: "8"
- board text added: "D14"
- board text added: "D15"
- board text added: "D16"
- board text added: "D17"
- board text added: "D18"
- board text added: "FREAKHAT"
- board text added: "GND"
- board text added: "RX"
- board text added: "SERIAL"
- board text added: "TX"
- board text added: "V1.0 • JANUARY 2026"
