File: MotorFreaker/FreakHat/_autosave-FreakHat.kicad_pcb (KiCad board)
At the start: 2 copper layers, 17 parts, among them J1 DIN-5, J10 Conn_01x05, J2 DIN-5, J4 Conn_01x05, J5 Conn_01x05, J6 Conn_01x05, J7 Conn_01x05, J8 Conn_01x05, J9 Conn_01x05, U1 74HC244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

Commit message: layout
Parts:
- turned RN1 to 180 degrees
Changed lines of the file:
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@@
 	(footprint "Resistor_THT:R_Array_SIP9"
 		(layer "F.Cu")
-		(at 94.488 36.322)
+		(at 94.488 36.322 180)
 		(descr "9-pin Resistor SIP pack")
 		(tags "R")
@@
 		)
 		(pad "1" thru_hole rect
-			(at 0 0)
+			(at 0 0 180)
 			(size 1.6 1.6)
 			(drill 0.8)
@@
 		)
 		(pad "2" thru_hole circle
-			(at 2.54 0)
+			(at 2.54 0 180)
 			(size 1.6 1.6)
 			(drill 0.8)
@@
 		)
 		(pad "3" thru_hole circle
-			(at 5.08 0)
+			(at 5.08 0 180)
 			(size 1.6 1.6)
 			(drill 0.8)
@@
 		)
 		(pad "4" thru_hole circle
-			(at 7.62 0)
+			(at 7.62 0 180)
 			(size 1.6 1.6)
 			(drill 0.8)
@@
 		)
 		(pad "5" thru_hole circle
-			(at 10.16 0)
+			(at 10.16 0 180)
 			(size 1.6 1.6)
 			(drill 0.8)
@@
 		)
 		(pad "6" thru_hole circle
-			(at 12.7 0)
+			(at 12.7 0 180)
 			(size 1.6 1.6)
 			(drill 0.8)
@@
 		)
 		(pad "7" thru_hole circle
-			(at 15.24 0)
+			(at 15.24 0 180)
 			(size 1.6 1.6)
 			(drill 0.8)
@@
 		)
 		(pad "8" thru_hole circle
-			(at 17.78 0)
+			(at 17.78 0 180)
 			(size 1.6 1.6)
 			(drill 0.8)
@@
 		)
 		(pad "9" thru_hole circle
-			(at 20.32 0)
+			(at 20.32 0 180)
 			(size 1.6 1.6)
 			(drill 0.8)
