File: MotorFreaker/FreakHat/FreakHat.kicad_sch (KiCad schematic)
At the start: 31 parts, among them J1 DIN-5, J10 Conn_01x05, J11 Barrel_Jack, J2 DIN-5, J3 Conn_01x05, J4 Conn_01x05, J5 Conn_01x05, J6 Conn_01x05, J7 Conn_01x05, J8 Conn_01x05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

Commit message: layout
Parts:
- removed J11: Barrel_Jack, symbol Connector:Barrel_Jack
- added J12, J13: Conn_01x02, Connector_JST:JST_XH_B2B-XH-AM_1x02_P2.50mm_Vertical, symbol Connector_Generic:Conn_01x02
- J10, J4, J5, J6, J7, J8, J9: footprint (none) -> Connector_JST:JST_XH_B5B-XH-AM_1x05_P2.50mm_Vertical
- U3: footprint (none) -> Package_DIP:DIP-8_W7.62mm_Socket
- U5: footprint SN7407N:DIP794W45P254L1969H508Q14 -> Package_DIP:DIP-14_W7.62mm_Socket
Connections:
- net +5V: no longer A1.VIN
- net +9V: now also A1.VIN
- net GND: now also J12.1 (Pin_1), J13.1 (Pin_1)
- net SW_1: now reaches A1.A2
- net SW_1: now also J12.2 (Pin_2)
- net SW_2: now reaches A1.A3
- net SW_2: now also J13.2 (Pin_2)
- no-connect marks 30 -> 28
Other:
- moved on the sheet: C3, C4, C5, U4

Commit message: midi
Parts:
- removed C6: 0.1uF, symbol Device:C
- removed D1: 1N4148, symbol Device:D_Schottky_Small
- removed J1, J2: DIN-5, FreakHat:DIN5_MIDI, symbol Connector:DIN-5
- removed R1, R2, R3: 220, symbol Device:R
- removed R4: 4.7K, symbol Device:R
- removed R5: 270, symbol Device:R
- removed RN1: 8 x 10K, Resistor_THT:R_Array_SIP9, symbol Device:R_Network08
- removed U3: 6N138, Package_DIP:DIP-8_W7.62mm_Socket, symbol Isolator:6N138
- removed U5: SN7407N, Package_DIP:DIP-14_W7.62mm_Socket, symbol SN7407N:SN7407N
- added J12: Conn_01x02, Connector_Molex:Molex_KK-254_AE-6410-02A_1x02_P2.54mm_Vertical, symbol Connector_Generic:Conn_01x02
- added J9: Conn_01x04, Connector_Molex:Molex_KK-254_AE-6410-04A_1x04_P2.54mm_Vertical, symbol Connector_Generic:Conn_01x04
- C1, C2, C5: footprint (none) -> Capacitor_THT:C_Disc_D3.4mm_W2.1mm_P2.50mm
- C3: footprint (none) -> Capacitor_THT:CP_Radial_D5.0mm_P2.00mm
- C4: footprint (none) -> Capacitor_THT:CP_Radial_D8.0mm_P3.50mm
- J1: renamed from J5; footprint Connector_JST:JST_XH_B5B-XH-AM_1x05_P2.50mm_Vertical -> Connector_Molex:Molex_KK-254_AE-6410-05A_1x05_P2.54mm_Vertical
- J10: renamed from J12; footprint Connector_JST:JST_XH_B2B-XH-AM_1x02_P2.50mm_Vertical -> Connector_Molex:Molex_KK-254_AE-6410-02A_1x02_P2.54mm_Vertical
- J11: renamed from J13; footprint Connector_JST:JST_XH_B2B-XH-AM_1x02_P2.50mm_Vertical -> Connector_Molex:Molex_KK-254_AE-6410-02A_1x02_P2.54mm_Vertical
- J2: renamed from J6; footprint Connector_JST:JST_XH_B5B-XH-AM_1x05_P2.50mm_Vertical -> Connector_Molex:Molex_KK-254_AE-6410-05A_1x05_P2.54mm_Vertical
- J3: renamed from J7; footprint Connector_JST:JST_XH_B5B-XH-AM_1x05_P2.50mm_Vertical -> Connector_Molex:Molex_KK-254_AE-6410-05A_1x05_P2.54mm_Vertical
- J4: renamed from J8; footprint Connector_JST:JST_XH_B5B-XH-AM_1x05_P2.50mm_Vertical -> Connector_Molex:Molex_KK-254_AE-6410-05A_1x05_P2.54mm_Vertical
- J5: renamed from J9; footprint Connector_JST:JST_XH_B5B-XH-AM_1x05_P2.50mm_Vertical -> Connector_Molex:Molex_KK-254_AE-6410-05A_1x05_P2.54mm_Vertical
- J6: renamed from J10; footprint Connector_JST:JST_XH_B5B-XH-AM_1x05_P2.50mm_Vertical -> Connector_Molex:Molex_KK-254_AE-6410-05A_1x05_P2.54mm_Vertical
- J7: renamed from J3; footprint (none) -> Connector_Molex:Molex_KK-254_AE-6410-05A_1x05_P2.54mm_Vertical
- J8: renamed from J4; footprint Connector_JST:JST_XH_B5B-XH-AM_1x05_P2.50mm_Vertical -> Connector_Molex:Molex_KK-254_AE-6410-05A_1x05_P2.54mm_Vertical
- SW1: footprint (none) -> Button_Switch_THT:SW_DIP_SPSTx02_Slide_9.78x7.26mm_W7.62mm_P2.54mm
Connections:
- net +5V: now also J9.2 (Pin_2)
- net CLK_1: now also U1.5 (2Y1); no longer U1.16 (1Y1)
- net CLK_2: now also U1.9 (2Y3); no longer U1.12 (1Y3)
- net CLK_3: now also U1.16 (1Y1); no longer U1.5 (2Y1)
- net CLK_4: now also U1.12 (1Y3); no longer U1.9 (2Y3)
- net CLK_5: now also U2.5 (2Y1); no longer U2.16 (1Y1)
- net CLK_6: now also U2.9 (2Y3); no longer U2.12 (1Y3)
- net CLK_7: now also U2.16 (1Y1); no longer U2.5 (2Y1)
- net CLK_8: now also U2.12 (1Y3); no longer U2.9 (2Y3)
- net CS_1: now also A1.D9; no longer A1.D2 (D2_INT0)
- net CS_2: now also A1.D5; no longer A1.D3 (D3_INT1)
- net CS_3: now also A1.D8; no longer A1.D4
- net CS_4: now also A1.D4; no longer A1.D5
- net CS_5: now also A1.D7; no longer A1.D6
- net CS_6: now also A1.D3 (D3_INT1); no longer A1.D7
- net CS_7: now also A1.D6; no longer A1.D8
- net CS_8: now also A1.D2 (D2_INT0); no longer A1.D9
- net DIP_1: now also A1.A0; no longer A1.A1
- net DIP_2: now also A1.A1; no longer A1.A0
- net DOUT_1: now also U1.3 (2Y0); no longer U1.18 (1Y0)
- net DOUT_2: now also U1.7 (2Y2); no longer U1.14 (1Y2)
- net DOUT_3: now also U1.18 (1Y0); no longer U1.3 (2Y0)
- net DOUT_4: now also U1.14 (1Y2); no longer U1.7 (2Y2)
- net DOUT_5: now also U2.3 (2Y0); no longer U2.18 (1Y0)
- net DOUT_6: now also U2.7 (2Y2); no longer U2.14 (1Y2)
- net DOUT_7: now also U2.18 (1Y0); no longer U2.3 (2Y0)
- net DOUT_8: now also U2.14 (1Y2); no longer U2.7 (2Y2)
- net GND: now also J12.1 (Pin_1), J9.1 (Pin_1)
- net at A1.D0 (D0/RX): now also J9.3 (Pin_3)
- net SW_3: now reaches A1.A4
- net SW_3: now also J12.2 (Pin_2)
- net at A1.D1 (D1/TX): now also J9.4 (Pin_4)
- no-connect marks 28 -> 16
