File: MotorFreaker/MotorFreaker/MotorFreaker.kicad_pcb (KiCad board)
At the start: 2 copper layers, 38.1 x 127 mm, 28 parts, among them J1 Conn_01x05, J10 OUT, J11 IN_V, J2 SPEED_POT, J3 POWER_POT, J4 EXTRA_POT, J5 CTRL_MODE, J6 BUTTON_MODE, J7 BUTTON, J8 LED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

Commit message: freaker
Parts:
- D2: value DIODE -> 1N5401
Changed lines of the file:
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@@
 			(pdf_back_fp_property_popups yes)
 			(pdf_metadata yes)
-			(pdf_single_document no)
+			(pdf_single_document yes)
 			(dxfpolygonmode yes)
 			(dxfimperialunits yes)
@@
 			(psnegative no)
 			(psa4output no)
-			(plot_black_and_white yes)
+			(plot_black_and_white no)
 			(sketchpadsonfab no)
 			(plotpadnumbers no)
@@
 			(crossoutdnponfab yes)
 			(subtractmaskfromsilk no)
-			(outputformat 1)
+			(outputformat 4)
 			(mirror no)
-			(drillshape 1)
+			(drillshape 0)
 			(scaleselection 1)
 			(outputdirectory "")
@@
 			(at 0 5.25 0)
 			(layer "F.Fab")
+			(hide yes)
 			(effects
 				(font
@@
 			)
 		)
-		(property "Value" "DIODE"
+		(property "Value" "1N5401"
 			(at 6.35 3.72 0)
 			(layer "F.Fab")
@@
 			(at 0 5.25 0)
 			(layer "F.Fab")
+			(hide yes)
 			(effects
 				(font
@@
 			(at 0 5.25 0)
 			(layer "F.Fab")
+			(hide yes)
 			(effects
 				(font
@@
 			(at 0 5.25 0)
 			(layer "F.Fab")
+			(hide yes)
 			(effects
 				(font
@@
 	)
 	(segment
-		(start 92.63 47.07)
-		(end 88.9 50.8)
-		(width 2.54)
-		(layer "F.Cu")
-		(net 8)
-	)
-	(segment
 		(start 92.63 33.71)
 		(end 92.63 41.91)
 		(width 2.54)
-		(layer "F.Cu")
+		(layer "B.Cu")
 		(net 8)
 	)
 	(segment
-		(start 92.63 41.91)
-		(end 92.63 47.07)
+		(start 92.63 47.07)
+		(end 88.9 50.8)
 		(width 2.54)
-		(layer "F.Cu")
+		(layer "B.Cu")
 		(net 8)
 	)
@@
 		(end 88.9 60.96)
 		(width 2.54)
-		(layer "F.Cu")
+		(layer "B.Cu")
+		(net 8)
+	)
+	(segment
+		(start 92.63 41.91)
+		(end 92.63 47.07)
+		(width 2.54)
+		(layer "B.Cu")
 		(net 8)
 	)
@@
 	)
 	(segment
-		(start 78.74 50.8)
-		(end 87.63 41.91)
-		(width 2.54)
-		(layer "F.Cu")
-		(net 17)
-	)
-	(segment
-		(start 76.2 49.53)
-		(end 76.2 50.8)
-		(width 2.54)
-		(layer "F.Cu")
-		(net 17)
-	)
-	(segment
 		(start 76.2 50.8)
 		(end 78.74 50.8)
 		(width 2.54)
-		(layer "F.Cu")
+		(layer "B.Cu")
 		(net 17)
 	)
 	(segment
-		(start 72.47 45.64)
-		(end 72.39 45.72)
+		(start 72.47 41.91)
+		(end 72.47 47.07)
 		(width 2.54)
-		(layer "F.Cu")
+		(layer "B.Cu")
 		(net 17)
 	)
 	(segment
-		(start 72.47 41.91)
-		(end 72.47 45.64)
+		(start 78.74 50.8)
+		(end 87.63 41.91)
 		(width 2.54)
-		(layer "F.Cu")
+		(layer "B.Cu")
 		(net 17)
 	)
 	(segment
-		(start 72.47 33.71)
-		(end 72.47 41.91)
+		(start 87.63 41.91)
+		(end 87.63 33.71)
 		(width 2.54)
-		(layer "F.Cu")
+		(layer "B.Cu")
 		(net 17)
 	)
 	(segment
-		(start 87.63 33.71)
-		(end 87.63 41.91)
+		(start 72.47 47.07)
+		(end 76.2 50.8)
 		(width 2.54)
-		(layer "F.Cu")
+		(layer "B.Cu")
 		(net 17)
 	)
 	(segment
-		(start 72.39 45.72)
-		(end 76.2 49.53)
+		(start 72.47 33.71)
+		(end 72.47 41.91)
 		(width 2.54)
-		(layer "F.Cu")
+		(layer "B.Cu")
 		(net 17)
 	)

Commit message: midi
Parts:
- removed REF** (x4): MountingHole_4.3mm_M4, MountingHole:MountingHole_4.3mm_M4
- removed REF**: Symbol_Attention_Triangle_8x7mm_Copper, Symbol:Symbol_Attention_Triangle_8x7mm_Copper
- added H1: MountingHole, MountingHole:MountingHole_3.5mm, F.Cu at (66.7, 19.1)
- added H2: MountingHole, MountingHole:MountingHole_3.5mm, F.Cu at (98.4, 19.1)
- added H3: MountingHole, MountingHole:MountingHole_3.5mm, F.Cu at (66.7, 139.7)
- added H4: MountingHole, MountingHole:MountingHole_3.5mm, F.Cu at (98.4, 139.7)
- J1: footprint Connector_JST:JST_XH_B5B-XH-AM_1x05_P2.50mm_Vertical -> Connector_Molex:Molex_KK-254_AE-6410-05A_1x05_P2.54mm_Vertical
- J2, J3, J4: footprint Connector_JST:JST_XH_B3B-XH-AM_1x03_P2.50mm_Vertical -> Connector_Molex:Molex_KK-254_AE-6410-03A_1x03_P2.54mm_Vertical
- J5, J6, J7, J8: footprint Connector_JST:JST_XH_B2B-XH-AM_1x02_P2.50mm_Vertical -> Connector_Molex:Molex_KK-254_AE-6410-02A_1x02_P2.54mm_Vertical
- R2: value R -> 270
Routing:
- net Net-(D2-K): track 41.9 -> 83.9 mm
- net Net-(D2-A): track 28.8 -> 57.6 mm
Other:
- board text added: "JANUARY 2026"
