File: MotorFreaker/MotorFreaker/MotorFreaker.kicad_sch (KiCad schematic)
At the start: 2 parts

Commit message: ups
Parts:
- added D?: D_Filled, symbol Device:D_Filled
- added D?: LED, symbol Device:LED
- added J1: Conn_02x03_Counter_Clockwise, symbol Connector_Generic:Conn_02x03_Counter_Clockwise
- added J?: POWER_POT, symbol Connector_Generic:Conn_01x03
- added J?: OUT_V, symbol Connector_Generic:Conn_01x02
- added J? (x2): BUTTON, symbol Connector_Generic:Conn_01x02
- added J?: SPEED_POT, symbol Connector_Generic:Conn_01x03
- added J?: OUT, symbol Connector_Generic:Conn_01x02
- added J?: LED, symbol Connector_Generic:Conn_01x02
- added Q?: NPN, symbol Simulation_SPICE:NPN
- added Q?: MOSFET, digikey-footprints:SOT-23-3, symbol MeowWolf_Devices:MOSFET
- added R? (x4): R, symbol Device:R
- gave numbers to parts that had none: 2
Connections:
- net MODE_C: now reaches U1.10 (PA3/AD3)
- net MODE_A: now reaches U1.11 (PA2/AD2)
- net POWER_POT: now reaches U1.12 (PA1/AD1)
- net SPEED_POT: now reaches U1.13 (AREF/PA0/AD0)
- net CS: now reaches U1.2 (XTAL1/PB0/D10)
- net RESET: now reaches U1.4 (~{RESET}/PB3)
- net RESET: now also J1.3 (Pin_3)
- net BUTTON: now reaches U1.5 (PB2/INT0/D8)
- net PWM: now reaches U1.6 (PA7/AD7)
- net PWM: now also R?.1, R?.1
- net DIN/MOSI: now reaches U1.7 (PA6/AD6)
- net DIN/MOSI: now also J1.5 (Pin_5)
- net MISO: now reaches U1.8 (PA5/AD5)
- net MISO: now also J1.1 (Pin_1)
- net CLK: now reaches U1.9 (PA4/AD4)
- net CLK: now also J1.2 (Pin_2)
- new net: D?.1 (K), J?.2 (Pin_2), J?.2 (Pin_2)
- new net: D?.2 (A), J?.1 (Pin_1), Q?.2 (D)
- new net: J?.1 (Pin_1), Q?.1 (C)
- new net: Q?.2 (B), R?.2
- new net: Q?.1 (G), R?.2, R?.2
- new net: J?.2 (Pin_2), R?.2
- new net +5V: J1.6 (Pin_6), R?.1
- new net GND: J1.4 (Pin_4), J?.1 (Pin_1), Q?.3 (E), Q?.3 (S), R?.1
Other:
- moved on the sheet: C1, U1

Commit message: module
Parts:
- removed D?: D_Filled, symbol Device:D_Filled
- removed D?: LED, symbol Device:LED
- removed J1: Conn_02x03_Counter_Clockwise, symbol Connector_Generic:Conn_02x03_Counter_Clockwise
- removed J?: POWER_POT, symbol Connector_Generic:Conn_01x03
- removed J?: OUT_V, symbol Connector_Generic:Conn_01x02
- removed J? (x2): BUTTON, symbol Connector_Generic:Conn_01x02
- removed J?: SPEED_POT, symbol Connector_Generic:Conn_01x03
- removed J?: OUT, symbol Connector_Generic:Conn_01x02
- removed J?: LED, symbol Connector_Generic:Conn_01x02
- removed Q?: NPN, symbol Simulation_SPICE:NPN
- removed Q?: MOSFET, digikey-footprints:SOT-23-3, symbol MeowWolf_Devices:MOSFET
- removed R? (x4): R, symbol Device:R
- removed U1: ATtiny84-20P, Package_DIP:DIP-14_W7.62mm, symbol MotorFreaker:ATtiny84-20P
- added C2: 10uF, symbol Device:C_Polarized_US
- added D1: 5V LED, symbol Device:D_Filled
- added D2: DIODE, symbol Device:D_Filled
- added J1: Conn_01x05, symbol Connector_Generic:Conn_01x05
- added J10: OUT, symbol Connector_Generic:Conn_01x02
- added J11: OUT_V, symbol Connector_Generic:Conn_01x02
- added J12: QT02ADP83H0000G, Amphenol_QT:QT02ADP83H0000G, symbol Amphenol_QT:QT02ADP83H0000G
- added J2: SPEED_POT, symbol Connector_Generic:Conn_01x03
- added J3: POWER_POT, symbol Connector_Generic:Conn_01x03
- added J4: EXTRA_POT, symbol Connector_Generic:Conn_01x03
- added J5: CTRL_MODE, symbol Connector_Generic:Conn_01x02
- added J6: BUTTON_MODE, symbol Connector_Generic:Conn_01x02
- added J7: BUTTON, symbol Connector_Generic:Conn_01x02
- added J8: LED, symbol Connector_Generic:Conn_01x02
- added J9: ICSP, Connector_IDC:IDC-Header_2x03_P2.54mm_Vertical, symbol Connector_Generic:Conn_02x03_Counter_Clockwise
- added Q1: NPN, symbol Simulation_SPICE:NPN
- added Q2: IRLZ44N, Package_TO_SOT_THT:TO-220-3_Vertical, symbol Transistor_FET:IRLZ44N
- added R1, R2: R, symbol Device:R
- added R3: 4.7K, symbol Device:R
- added R4: 10K, symbol Device:R
- added R5: 220, symbol Device:R
- added U2: ATtiny84, Package_DIP:DIP-14_W7.62mm, symbol MotorFreaker:ATtiny84-20P
- C1: value C -> 0.1uF
Connections:
- net +5V: now also C1.1, C2.1, J1.2 (Pin_2), J2.3 (Pin_3), J3.3 (Pin_3), J4.3 (Pin_3), J9.6 (Pin_6), R1.1, R2.2, U2.1 (VCC)
- net BUTTON: now also J7.2 (Pin_2), U2.5 (PB2/INT0/D8)
- net CLK: now also J1.4 (Pin_4), J9.2 (Pin_2), U2.9 (PA4/AD4)
- net CS: now also J1.3 (Pin_3), U2.2 (XTAL1/PB0/D10)
- net GND: now also C1.2, C2.2, D1.1 (K), J1.1 (Pin_1), J11.1 (Pin_1), J2.1 (Pin_1), J3.1 (Pin_1), J4.1 (Pin_1), J5.1 (Pin_1), J6.1 (Pin_1), J7.1 (Pin_1), J9.4 (Pin_4), Q1.3 (E), Q2.3 (S), R4.1, U2.14 (GND)
- net MISO: now also J9.1 (Pin_1), U2.8 (PA5/AD5)
- net POWER_POT: now also J3.2 (Pin_2), U2.12 (PA1/AD1)
- net PWM: now also R3.1, R4.2, R5.1, U2.6 (PA7/AD7)
- net RESET: now also J9.3 (Pin_3), U2.4 (~{RESET}/PB3)
- net SPEED_POT: now also J2.2 (Pin_2), U2.13 (AREF/PA0/AD0)
- new net: Q2.1 (G), R5.2
- new net: D2.2 (A), J10.1 (Pin_1), Q2.2 (D)
- new net: Q1.2 (B), R3.2
- new net: J8.1 (Pin_1), Q1.1 (C)
- new net: J8.2 (Pin_2), R2.1
- new net: D2.1 (K), J10.2 (Pin_2), J11.2 (Pin_2)
- new net: D1.2 (A), R1.2
- new net BUTTON_MODE: J6.2 (Pin_2), U2.3 (XTAL2/PB1/D9)
- new net CTRL_MODE: J5.2 (Pin_2), U2.10 (PA3/AD3)
- new net DIN: J1.5 (Pin_5), J9.5 (Pin_5), U2.7 (PA6/AD6)
- new net EXTRA_POT: J4.2 (Pin_2), U2.11 (PA2/AD2)

Commit message: pcb
Parts:
- removed D1: 5V LED, symbol Device:D_Filled
- removed J10: OUT, symbol Connector_Generic:Conn_01x02
- removed J11: OUT_V, symbol Connector_Generic:Conn_01x02
- removed J12: QT02ADP83H0000G, Amphenol_QT:QT02ADP83H0000G, symbol Amphenol_QT:QT02ADP83H0000G
- removed J9: ICSP, Connector_IDC:IDC-Header_2x03_P2.54mm_Vertical, symbol Connector_Generic:Conn_02x03_Counter_Clockwise
- added D1: 5V, LED_THT:LED_D3.0mm, symbol Device:LED_Filled
- added J10: OUT, Amphenol_QT:QT02ADP83H0000G, symbol Connector_Generic:Conn_01x04
- added J11: IN_V, Amphenol_QT:QT02ADP83H0000G, symbol Connector_Generic:Conn_01x04
- added J9: ICSP, Connector_PinHeader_2.54mm:PinHeader_2x03_P2.54mm_Vertical, symbol Connector_Generic:Conn_02x03_Odd_Even
- C1: footprint (none) -> Capacitor_THT:C_Disc_D3.4mm_W2.1mm_P2.50mm
- C2: footprint (none) -> Capacitor_THT:CP_Radial_D5.0mm_P2.00mm
- D2: footprint (none) -> Diode_THT:D_DO-201AD_P12.70mm_Horizontal
- J1: footprint (none) -> Connector_JST:JST_XH_B5B-XH-AM_1x05_P2.50mm_Vertical
- J2, J3, J4: footprint (none) -> Connector_JST:JST_XH_B3B-XH-AM_1x03_P2.50mm_Vertical
- J5, J6, J7, J8: footprint (none) -> Connector_JST:JST_XH_B2B-XH-AM_1x02_P2.50mm_Vertical
- Q1: footprint (none) -> Package_TO_SOT_THT:TO-92L_Inline_Wide
- R1: value R -> 1.5K; footprint (none) -> Resistor_THT:R_Axial_DIN0207_L6.3mm_D2.5mm_P7.62mm_Horizontal
- R2, R3, R4, R5: footprint (none) -> Resistor_THT:R_Axial_DIN0207_L6.3mm_D2.5mm_P7.62mm_Horizontal
Connections:
- net +5V: now also J9.2 (Pin_2)
- net CLK: now also J1.3 (Pin_3), J9.3 (Pin_3); no longer J1.4 (Pin_4)
- net CS: now also J1.5 (Pin_5), U2.10 (PA3/AD3); no longer J1.3 (Pin_3), U2.2 (XTAL1/PB0/D10)
- net CTRL_MODE: now also U2.2 (XTAL1/PB0/D10); no longer U2.10 (PA3/AD3)
- net DIN: now also J1.4 (Pin_4), J9.4 (Pin_4); no longer J1.5 (Pin_5)
- net GND: now also D1.1 (K), J11.1 (Pin_1), J11.2 (Pin_2), J9.6 (Pin_6)
- net MISO: now also J9.1 (Pin_1)
- net RESET: now also J9.5 (Pin_5)
- net at D2.2 (A), Q2.2 (D): now also J10.1 (Pin_1), J10.2 (Pin_2)
- net at D2.1 (K): now also J10.3 (Pin_3), J10.4 (Pin_4), J11.3 (Pin_3), J11.4 (Pin_4)
- net at R1.2: now also D1.2 (A)
Other:
- moved on the sheet: D2, J2, J3, J4, J5, J6, J7, J8, R1

Commit message: freaker
Parts:
- D2: value DIODE -> 1N5401
Changed lines of the file:
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@@
 			)
 		)
-		(property "Value" "DIODE"
+		(property "Value" "1N5401"
 			(at 190.5 129.5399 90)
 			(effects

Commit message: layout
Parts:
- R2: value R -> 270
Changed lines of the file:
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@@
 			)
 		)
-		(property "Value" "R"
+		(property "Value" "270"
 			(at 190.5 106.6799 0)
 			(effects

Commit message: midi
Parts:
- added H1, H2, H3, H4: MountingHole, MountingHole:MountingHole_3.5mm, symbol Mechanical:MountingHole
- J1: footprint Connector_JST:JST_XH_B5B-XH-AM_1x05_P2.50mm_Vertical -> Connector_Molex:Molex_KK-254_AE-6410-05A_1x05_P2.54mm_Vertical
- J2, J3, J4: footprint Connector_JST:JST_XH_B3B-XH-AM_1x03_P2.50mm_Vertical -> Connector_Molex:Molex_KK-254_AE-6410-03A_1x03_P2.54mm_Vertical
- J5, J6, J7, J8: footprint Connector_JST:JST_XH_B2B-XH-AM_1x02_P2.50mm_Vertical -> Connector_Molex:Molex_KK-254_AE-6410-02A_1x02_P2.54mm_Vertical
